Commit message: aggiunti limiti di giunto

File: simulator_edo/urdf/edo_sim.urdf (robot description, URDF)
Before this commit: robot edo_sim, 7 links, 6 joints
Joints:
- joint joint_1: limit (none) -> lower=-3.14 upper=3.14 effort=5000 velocity=0.6632; type continuous -> revolute
- joint joint_2: limit (none) -> lower=-1.972 upper=1.972 effort=5000 velocity=0.6632; type continuous -> revolute
- joint joint_3: limit (none) -> lower=-1.972 upper=1.972 effort=5000 velocity=0.6632; type continuous -> revolute
- joint joint_4: limit (none) -> lower=-3.14 upper=3.14 effort=5000 velocity=0.97738; type continuous -> revolute
- joint joint_5: limit (none) -> lower=-1.815 upper=1.815 effort=5000 velocity=0.97738; type continuous -> revolute
- joint joint_6: limit (none) -> lower=-47.1238 upper=47.1238 effort=5000 velocity=0.97738; type continuous -> revolute

Commit message: Started conversion to 3 joints

File: simulator_edo/urdf/edo_sim.urdf (robot description, URDF)
Before this commit: robot edo_sim, 7 links, 6 joints
Joints:
- joint joint_4: limit lower=-3.14 upper=3.14 effort=5000 velocity=0.97738 -> (none); type revolute -> fixed
- joint joint_5: limit lower=-1.815 upper=1.815 effort=5000 velocity=0.97738 -> (none); type revolute -> fixed
- joint joint_6: limit lower=-47.1238 upper=47.1238 effort=5000 velocity=0.97738 -> (none); type revolute -> fixed
