Commit message: Added drag and gravity,  moved COM to joint origin

File: simulator_edo/urdf/edo_sim_nuove_inerzie.urdf (robot description, URDF)
Before this commit: robot edo_sim, 7 links, 6 joints
Joints:
- joint joint_1: limit lower=-3.14 upper=3.14 effort=5000 velocity=0.6632 -> (none)
- joint joint_2: limit lower=-1.972 upper=1.972 effort=5000 velocity=0.6632 -> (none)
- joint joint_3: limit lower=-1.972 upper=1.972 effort=5000 velocity=0.6632 -> (none)

Commit message: bugfix

File: simulator_edo/urdf/edo_sim_nuove_inerzie.urdf (robot description, URDF)
Before this commit: robot edo_sim, 7 links, 6 joints
Joints:
- joint joint_2: type continuous -> fixed
- joint joint_3: type continuous -> fixed

Commit message: bugfixes

File: simulator_edo/urdf/edo_sim_nuove_inerzie.urdf (robot description, URDF)
Before this commit: robot edo_sim, 7 links, 6 joints
Joints:
- joint joint_1: limit lower=-3.14 upper=3.14 effort=5000 velocity=0.6632 -> (none)
- joint joint_2: limit lower=-1.972 upper=1.972 effort=5000 velocity=0.6632 -> (none); type fixed -> continuous
- joint joint_3: limit lower=-1.972 upper=1.972 effort=5000 velocity=0.6632 -> (none); type fixed -> continuous
